Commit message: fixed gazebo error

File: table_arm/table_arm/urdf/table_arm.transmission.xacro (robot description, xacro)
@@ -1,10 +1,5 @@
 <?xml version="1.0"?>
-<robot>
+<robot xmlns:xacro="http://www.ros.org/wiki/xacro">
   <!-- parses the transmission tags and loads the appropriate hardware interfaces and controller manager -->
-  <gazebo>
-    <plugin name="gazebo_ros_control" filename="libgazebo_ros_control.so">
-      <robotNamespace>/robot</robotNamespace>
-      <robotSimType>gazebo_ros_control/DefaultRobotHWSim</robotSimType>
-    </plugin>
   <!-- <robot xmlns:xacro="http://www.ros.org/wiki/xacro">
   <xacro:macro name="table_arm_transmission" params="side"> -->
@@ -70,4 +65,3 @@
     </actuator>
   </transmission>
-  </gazebo>
 </robot>

File: table_arm/table_arm/urdf/table_arm.xacro (robot description, xacro)
@@ -6,5 +6,5 @@
   name="table_arm" xmlns:xacro="http://www.ros.org/wiki/xacro">
   <!-- <xacro:include filename="$(find table_arm)/urdf/controller.gazebo" /> -->
-  <xacro:include filename="$(find table_arm)/urdf/description.gazebo" />
+  <xacro:include filename="$(find table_arm)/urdf/table_arm.gazebo.xacro" />
   <xacro:include filename="$(find table_arm)/urdf/table_arm.transmission.xacro" />
   <link name="world"/>
@@ -25,10 +25,10 @@
         value="1.12509149890152" />
       <inertia
-        ixx="0.00101434409151112"
-        ixy="-1.04880216285518E-06"
-        ixz="2.00480977970094E-07"
-        iyy="0.00103853740225625"
-        iyz="1.41989902783292E-06"
-        izz="0.00175265916240766" />
+        ixx="0.1"
+        ixy="0"
+        ixz="0"
+        iyy="0.1"
+        iyz="0"
+        izz="0.1" />
     </inertial>
     <visual>
@@ -65,10 +65,10 @@
         value="1.18180242682421" />
       <inertia
-        ixx="0.000885516457055022"
-        ixy="-4.93627366915009E-06"
-        ixz="-2.91116322104174E-06"
-        iyy="0.00138668286939693"
-        iyz="1.56769429304993E-06"
-        izz="0.00115252171660378" />
+        ixx="0.1"
+        ixy="0"
+        ixz="0"
+        iyy="0.1"
+        iyz="0"
+        izz="0.1" />
     </inertial>
     <visual>
@@ -123,10 +123,10 @@
         value="0.742154760471324" />
       <inertia
-        ixx="0.000383418033802214"
-        ixy="1.95626085431396E-06"
-        ixz="5.52016092099987E-06"
-        iyy="0.000519769983990921"
-        iyz="-4.81334906226082E-06"
-        izz="0.000422634222999281" />
+        ixx="0.1"
+        ixy="0"
+        ixz="0"
+        iyy="0.1"
+        iyz="0"
+        izz="0.1" />
     </inertial>
     <visual>
@@ -181,10 +181,10 @@
         value="0.806964917043645" />
       <inertia
-        ixx="0.000369652873297802"
-        ixy="-1.52204773385423E-06"
-        ixz="1.20034094378975E-06"
-        iyy="0.000335533295104123"
-        iyz="-1.1515591101845E-05"
-        izz="0.000394955086054961" />
+        ixx="0.1"
+        ixy="0"
+        ixz="0"
+        iyy="0.1"
+        iyz="0"
+        izz="0.1" />
     </inertial>
     <visual>
@@ -214,5 +214,5 @@
   <joint
     name="joint_3"
-    type="continuous">
+    type="revolute">
     <origin
       xyz="0 -0.1445 -0.00749999999998746"
@@ -224,4 +224,9 @@
     <axis
       xyz="0 0 -1" />
+    <limit
+      lower="-3.14"
+      upper="3.14"
+      effort="1000"
+      velocity="6.5" />
   </joint>
   <link
@@ -234,10 +239,10 @@
         value="0.566102198606674" />
       <inertia
-        ixx="0.000260590319873162"
-        ixy="-5.08487877698499E-05"
-        ixz="-3.4003226615359E-06"
-        iyy="0.000284217607682232"
-        iyz="-5.22728155265439E-06"
-        izz="0.000225229416725362" />
+        ixx="0.1"
+        ixy="0"
+        ixz="0"
+        iyy="0.1"
+        iyz="0"
+        izz="0.1" />
     </inertial>
     <visual>
@@ -292,10 +297,10 @@
         value="0.468596922084729" />
       <inertia
-        ixx="0.000163486477461417"
-        ixy="-1.12447617071923E-09"
-        ixz="-3.05692009732978E-07"
-        iyy="0.000226300679826748"
-        iyz="-1.3266635516296E-05"
-        izz="0.000178272106720262" />
+        ixx="0.1"
+        ixy="0"
+        ixz="0"
+        iyy="0.1"
+        iyz="0"
+        izz="0.1" />
     </inertial>
     <visual>
@@ -325,5 +330,5 @@
   <joint
     name="joint_5"
-    type="continuous">
+    type="revolute">
     <origin
       xyz="-0.118793939239341 0.0671751442127215 0.00399999999999767"
@@ -335,4 +340,9 @@
     <axis
       xyz="0 0 -1" />
+    <limit
+      lower="-3.14"
+      upper="3.14"
+      effort="1000"
+      velocity="6.5" />
   </joint>
   <link
@@ -345,10 +355,10 @@
         value="0.410187464873175" />
       <inertia
-        ixx="0.000155615505356158"
-        ixy="-1.61032292748035E-05"
-        ixz="-6.67491379603911E-06"
-        iyy="0.000180111157412533"
-        iyz="1.27737173899181E-05"
-        izz="0.000106091737904499" />
+        ixx="0.1"
+        ixy="0"
+        ixz="0"
+        iyy="0.1"
+        iyz="0"
+        izz="0.1" />
     </inertial>
     <visual>
